Commit message: new kinetic

File: phantomx_reactor_arm_description/robots/phantomx_reactor_arm_no_wrist.urdf.xacro (robot description, xacro)
@@ -11,5 +11,5 @@
 		</visual>
 	</link>
-	<xacro:phantomx_reactor_no_wrist prefix="arm_" parent="base_footprint">
+	<xacro:phantomx_reactor_no_wrist prefix="" parent="base_footprint">
 		<origin xyz="0 0 0" rpy="0 0 0" />
 	</xacro:phantomx_reactor_no_wrist>

File: phantomx_reactor_arm_description/urdf/phantomx_reactor_no_wrist.urdf.xacro (robot description, xacro)
@@ -10,4 +10,6 @@
 	<xacro:property name="joint_4_upper_limit" value="${PI/2}"/>
 	<xacro:property name="joint_4_lower_limit" value="-${PI/2}"/>
+	<xacro:property name="gripper_joint_upper_limit" value="0.0"/>
+	<xacro:property name="gripper_joint_lower_limit" value="0.03"/>
 	<xacro:macro name="phantomx_reactor_no_wrist" params="parent prefix *origin">
 		<joint name="${prefix}base_joint" type="fixed">
@@ -40,13 +42,13 @@
 			</collision>
 		</link>
-		<!-- JOINT 1 -->
-		<joint name="${prefix}1_joint" type="revolute">
+		<!-- SHOULDER YAW -->
+		<joint name="${prefix}shoulder_yaw_joint" type="revolute">
 			<origin xyz="0 0 0.081" rpy="0 0 0" />
 			<parent link="${prefix}base_link" />
-			<child link="${prefix}1_link" />
+			<child link="${prefix}shoulder_link" />
 			<axis xyz="0 0 1" />
 			<limit effort="1.5" velocity="6.178465545" lower="-3.141593" upper="3.141593" />
 		</joint>
-		<link name="${prefix}1_link">
+		<link name="${prefix}shoulder_link">
 			<inertial>
 			  <origin xyz="5.5296E-07 0.00048339 0.0026355" rpy="0 0 0" />
@@ -72,13 +74,13 @@
 			</collision>
 		</link>
-		<!-- JOINT 2 -->
-		<joint name="${prefix}2_joint" type="revolute">
+		<!-- SHOULDER PITCH -->
+		<joint name="${prefix}shoulder_pitch_joint" type="revolute">
 			<origin xyz="0 0 0.0265" rpy="${PI/2} 0 0" />
-			<parent link="${prefix}1_link" />
-			<child link="${prefix}2_link" />
+			<parent link="${prefix}shoulder_link" />
+			<child link="${prefix}bicep_link" />
 			<axis xyz="0 0 -1" />
 			<limit effort="3.0" velocity="6.178465545" lower="${joint_2_lower_limit}" upper="${joint_2_upper_limit}" />
 		</joint>
-		<link name="${prefix}2_link">
+		<link name="${prefix}bicep_link">
 			<inertial>
 			  <origin xyz="-0.079312 0.00175 0.0073486" rpy="-${PI/2} 0 -${PI/2}" />
@@ -105,13 +107,13 @@
 			</collision>
 	  </link>
-	  <!-- JOINT 3 -->
-	  <joint name="${prefix}3_joint"	type="revolute">
+	   <!-- ELBOW PITCH-->
+	  <joint name="${prefix}elbow_pitch_joint"	type="revolute">
 		<origin xyz="0.0385 0.1445 0.0" rpy="0 0 0" />
-		<parent link="${prefix}2_link" />
-		<child link="${prefix}3_link" />
+		<parent link="${prefix}bicep_link" />
+		<child link="${prefix}forearm_link" />
 		<axis xyz="0 0 1" />
 		<limit effort="3.0" velocity="6.178465545" lower="${joint_3_lower_limit}" upper="${joint_3_upper_limit}"/>
 	  </joint>
-	  <link name="${prefix}3_link">
+	  <link name="${prefix}forearm_link">
 		<inertial>
 		  <origin xyz="0.0851888339312843 0.00136288621406396 -0.000141576344087929" rpy="-${PI/2} 0 0" />
@@ -137,13 +139,13 @@
 		</collision>
 	  </link>
-	  <!-- JOINT 4 -->
-	  <joint name="${prefix}4_joint"	type="revolute">
+	  <!-- WRIST PITCH-->
+	  <joint name="${prefix}wrist_pitch_joint"	type="revolute">
 		<origin xyz="0.1535 0 0" rpy="0 0 0" />
-		<parent link="${prefix}3_link" />
-		<child link="${prefix}4_link" />
+		<parent link="${prefix}forearm_link" />
+		<child link="${prefix}wrist_1_link" />
 		<axis xyz="0 0 1" />
 		<limit effort="1.5" velocity="6.178465545" lower="${joint_4_lower_limit}" upper="${joint_4_upper_limit}" />
 	  </joint>
-	  <link name="${prefix}4_link">
+	  <link name="${prefix}wrist_1_link">
 		<inertial>
 		  <origin xyz="0.0426453655090486 0.0017494960392062 0.00984847105297723" rpy="-${PI/2} 0 0" />
@@ -170,141 +172,91 @@
 	  </link>
 	  <!-- GRIPPER -->
-	   <joint name="${prefix}gripper_joint" type="fixed">
-		<origin xyz="0.07289 0.00175 0" rpy="${PI/2} 0 0" />
-		<parent link="${prefix}4_link" />
-		<child link="${prefix}gripper_link" />
-		<axis xyz="0 0 0" />
-	  </joint>
-	  <link name="${prefix}gripper_link">
-		<inertial>
-		  <origin xyz="0.0091884 -7.3309E-13 -3.4513E-05" rpy="0 0 0" />
-		  <mass value="0.02487" />
-		  <inertia  ixx="1.5997E-05" ixy="1.6551E-16" ixz="8.3911E-09"
-					iyy="7.3918E-06" iyz="-2.7145E-16"
-					izz="1.5931E-05" />
-		</inertial>
-		<visual>
-		  <origin xyz="0 0 0" rpy="0 0 0" />
-		  <geometry>
-			<mesh filename="package://phantomx_reactor_arm_description/meshes/gripper_link.STL" />
-		  </geometry>
-		  <material name="">
-			<color rgba="0.25098 0.25098 0.25098 1" />
-		  </material>
-		</visual>
-		<collision>
-		  <origin xyz="0 0 0" rpy="0 0 0" />
-		  <geometry>
-			<mesh filename="package://phantomx_reactor_arm_description/meshes/gripper_link_hull.STL" />
-		  </geometry>
-		</collision>
-	  </link>
-	  <!--
-	  <link	name="wrist_2">
-		<inertial>
-		  <origin
-			xyz="0.022349 -5.4754E-07 0.0089164"
-			rpy="0 0 0" />
-		  <mass
-			value="0.055706" />
-		  <inertia
-			ixx="1.5957E-05"
-			ixy="2.0952E-10"
-			ixz="3.3629E-06"
-			iyy="2.1196E-05"
-			iyz="-2.4643E-10"
-			izz="1.4482E-05" />
-		</inertial>
-		<visual>
-		  <origin
-			xyz="0 0 0"
-			rpy="0 0 0" />
-		  <geometry>
-			<mesh
-			  filename="package://phantomx_reactor_arm_description/meshes/wrist_2.STL" />
-		  </geometry>
-		  <material
-			name="">
-			<color
-			  rgba="0.25098 0.25098 0.25098 1" />
-		  </material>
-		</visual>
-		<collision>
-		  <origin
-			xyz="0 0 0"
-			rpy="0 0 0" />
-		  <geometry>
-			<mesh
-			  filename="package://phantomx_reactor_arm_description/meshes/wrist_2_hull.STL" />
-		  </geometry>
-		</collision>
-	  </link>
-	  <joint name="wrist_roll"type="revolute">
-		<origin
-		  xyz="0.071 0.00175 0"
-		  rpy="0 0 0" />
-		<parent
-		  link="wrist_1" />
-		<child
-		  link="wrist_2" />
-		<axis
-		  xyz="1 0 0" />
-		<limit
-		  effort="1.5"
-		  velocity="6.178465545"
-		  lower="-3.141593"
-		  upper="3.141593" />
-	  </joint>
-	  <link name="gripper_link">
-		<inertial>
-		  <origin
-			xyz="0.0091884 -7.3309E-13 -3.4513E-05"
-			rpy="0 0 0" />
-		  <mass
-			value="0.02487" />
-		  <inertia
-			ixx="1.5997E-05"
-			ixy="1.6551E-16"
-			ixz="8.3911E-09"
-			iyy="7.3918E-06"
-			iyz="-2.7145E-16"
-			izz="1.5931E-05" />
-		</inertial>
-		<visual>
-		  <origin
-			xyz="0 0 0"
-			rpy="0 0 0" />
-		  <geometry>
-			<mesh
-			  filename="package://phantomx_reactor_arm_description/meshes/gripper_link.STL" />
-		  </geometry>
-		  <material
-			name="">
-			<color
-			  rgba="0.25098 0.25098 0.25098 1" />
-		  </material>
-		</visual>
-		<collision>
-		  <origin
-			xyz="0 0 0"
-			rpy="0 0 0" />
-		  <geometry>
-			<mesh
-			  filename="package://phantomx_reactor_arm_description/meshes/gripper_link_hull.STL" />
-		  </geometry>
-		</collision>
-	  </link>
-	  <joint name="gripper_joint" type="fixed">
-		<origin
-		  xyz="0.04789 0 0"
-		  rpy="0 0 0" />
-		<parent
-		  link="wrist_2" />
-		<child
-		  link="gripper_link" />
-		<axis
-		  xyz="0 0 0" />
-	  </joint>
-	  -->
+		<joint name="${prefix}gripper_guide_joint" type="fixed">
+			<origin xyz="0.07289 0.00175 0" rpy="${PI/2} 0 0" />
+			<parent link="${prefix}wrist_1_link" />
+			<child link="${prefix}gripper_guide_link" />
+			<axis xyz="0 0 1" />
+			<limit effort="1.5" velocity="6.178465545" lower="0" upper="1.57"/>
+		</joint>
+		<link name="${prefix}gripper_guide_link">
+			<inertial>
+				<origin xyz="0.0091884 -7.3309E-13 -3.4513E-05" rpy="0 0 0" />
+				<mass value="0.02487" />
+				<inertia ixx="1.5997E-05" ixy="1.6551E-16" ixz="8.3911E-09" iyy="7.3918E-06" iyz="-2.7145E-16" izz="1.5931E-05" />
+			</inertial>
+			<visual>
+				<origin xyz="0 0 0" rpy="1.57 3.14 1.57" />
+				<geometry>
+					<mesh filename="package://phantomx_reactor_arm_description/meshes/Guide_Rail_Fixed_Centered.stl" scale="0.01 0.01 0.01" />
+				</geometry>
+				<material name="">
+					<color rgba="0.25098 0.25098 0.25098 1" />
+				</material>
+			</visual>
+			<collision>
+				<origin xyz="0 0 0" rpy="1.57 3.14 1.57" />
+				<geometry>
+					<mesh filename="package://phantomx_reactor_arm_description/meshes/Guide_Rail_Fixed_Centered.stl" scale="0.01 0.01 0.01" />
+				</geometry>
+			</collision>
+		</link>
+		<joint name="${prefix}gripper_revolute_joint" type="revolute">
+			 <origin xyz = "0 0 0" rpy="0 ${PI/2} 0" />
+			 <parent link="${prefix}gripper_guide_link" />
+			 <child link="${prefix}gripper_aux_link" />
+			 <axis xyz="0 0 1" />
+			 <limit lower="-${PI}" upper="${PI}" effort="0" velocity="0.5" />
+        </joint>
+        <link name="${prefix}gripper_aux_link">
+		</link>
+		<joint name="${prefix}gripper_right_joint" type="prismatic">
+			<origin xyz="0.0202 0 0"   rpy="0 0 0" />
+			<parent link="${prefix}gripper_guide_link" />
+			<child link="${prefix}gripper_right_link" />
+			<axis xyz="0 1 0" />
+			<limit effort="1.5" velocity="6.178465545" lower="${gripper_joint_lower_limit}" upper="${gripper_joint_upper_limit}" />
+		</joint>
+		<link name="${prefix}gripper_right_link">
+			<visual>
+				<origin xyz="0 0.010 0" rpy="-1.57 -1.57 0" />
+				<geometry>
+					<mesh filename="package://phantomx_reactor_arm_description/meshes/Gripper_Hand_Fixed_Centered.stl" scale="0.01 0.01 0.01" />
+				</geometry>
+				<material name="">
+					<color rgba="0.25098 0.25098 0.25098 1" />
+				</material>
+			</visual>
+			<collision>
+				<origin xyz="0 0.010 0" rpy="-1.57 -1.57 0" />
+				<geometry>
+					<mesh filename="package://phantomx_reactor_arm_description/meshes/Gripper_Hand_Fixed_Centered.stl" scale="0.01 0.01 0.01" />
+				</geometry>
+			</collision>
+		</link>
+		<joint name="${prefix}gripper_left_joint" type="prismatic">
+			<origin xyz="0.0202 0 0" rpy="0 0 0" />
+			<parent link="${prefix}gripper_guide_link" />
+			<child link="${prefix}gripper_left_link" />
+			<axis xyz="0 1 0" />
+			<limit effort="1.5" velocity="6.178465545"  lower="-1.9" upper="0" />
+			<mimic joint="${prefix}gripper_right_joint" multiplier="-1.0"/>
+		</joint>
+		<link name="${prefix}gripper_left_link">
+			<visual>
+				<origin xyz="0 -0.010 0" rpy="1.57 1.57 0" />
+				<geometry>
+					<mesh filename="package://phantomx_reactor_arm_description/meshes/Gripper_Hand_Fixed_Centered.stl" scale="0.01 0.01 0.01" />
+				</geometry>
+				<material name="">
+					<color rgba="0.25098 0.25098 0.25098 1" />
+				</material>
+			</visual>
+			<collision>
+				<origin xyz="0 -0.010 0" rpy="1.57 1.57 0" />
+				<geometry>
+					<mesh filename="package://phantomx_reactor_arm_description/meshes/Gripper_Hand_Fixed_Centered.stl" scale="0.01 0.01 0.01" />
+				</geometry>
+			</collision>
+		</link>
 	</xacro:macro>
 </robot>
